Commit message: Rewrite gait: Cartesian trot with exact URDF IK, cmd_vel teleop, Gazebo test
- Package is now twist_2_0_description (replaces the earlier twist_walker layout)
- kinematics.py: leg FK/IK taken directly from the URDF, kept within soft limits
- gait.py: velocity-driven trot/crawl, centred foot placement, smooth start/stop,
  commands scaled to what the legs and servos can reach
- cmd_vel_gait / walk_gait: sim time, stand-up from /joint_states, live params,
  cmd_timeout 0 keeps the last command (works with teleop_twist_keyboard)
- gz_ros2_control position_proportional_gain 1.0 (default 0.1 lagged every step)
- OdometryPublisher plugin, ground truth bridged to /odom
- gait_test: automated closed-loop walking check in Gazebo; unit tests
- README with full setup / run / test commands; robot details in docs/ROBOT.md

Co-Authored-By: Claude Opus 5.5 <noreply@anthropic.com>

File: urdf/twist_2_0.urdf (robot description, URDF)
Before this commit: robot twist_2_0, 13 links, 12 joints
Links:
- link FL_hip: mass 0.01460 -> 0.01994; geometry collision mesh filename=package://twist_2_0_description/meshes/collision/FL_hip_0.s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; collision mesh filename=package://twist_2_0_description/meshes/collision/FL_hip_1.s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
- link FL_shin: mass 0.03421 -> 0.03688; geometry collision mesh filename=package://twist_2_0_description/meshes/collision/FL_shin_0.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; collision mesh filename=package://twist_2_0_description/meshes/collision/FL_shin_1.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
- link FL_thigh: mass 0.11726 -> 0.12481; geometry collision mesh filename=package://twist_2_0_description/meshes/collision/FL_thigh_0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; collision mesh filename=package://twist_2_0_description/meshes/collision/FL_thigh_1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
- link FR_hip: mass 0.01460 -> 0.01994; geometry collision mesh filename=package://twist_2_0_description/meshes/collision/FR_hip_0.s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; collision mesh filename=package://twist_2_0_description/meshes/collision/FR_hip_1.s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
- link FR_shin: mass 0.03421 -> 0.03688; geometry collision mesh filename=package://twist_2_0_description/meshes/collision/FR_shin_0.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; collision mesh filename=package://twist_2_0_description/meshes/collision/FR_shin_1.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
- link FR_thigh: mass 0.11726 -> 0.12481; geometry collision mesh filename=package://twist_2_0_description/meshes/collision/FR_thigh_0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; collision mesh filename=package://twist_2_0_description/meshes/collision/FR_thigh_1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
- link RL_hip: mass 0.01460 -> 0.01994; geometry collision mesh filename=package://twist_2_0_description/meshes/collision/RL_hip_0.s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; collision mesh filename=package://twist_2_0_description/meshes/collision/RL_hip_1.s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
- link RL_shin: mass 0.03421 -> 0.03688; geometry collision mesh filename=package://twist_2_0_description/meshes/collision/RL_shin_0.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; collision mesh filename=package://twist_2_0_description/meshes/collision/RL_shin_1.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
- link RL_thigh: mass 0.11726 -> 0.12481; geometry collision mesh filename=package://twist_2_0_description/meshes/collision/RL_thigh_0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; collision mesh filename=package://twist_2_0_description/meshes/collision/RL_thigh_1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
- link RR_hip: mass 0.01460 -> 0.01994; geometry collision mesh filename=package://twist_2_0_description/meshes/collision/RR_hip_0.s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; collision mesh filename=package://twist_2_0_description/meshes/collision/RR_hip_1.s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
- link RR_shin: mass 0.03421 -> 0.03688; geometry collision mesh filename=package://twist_2_0_description/meshes/collision/RR_shin_0.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; collision mesh filename=package://twist_2_0_description/meshes/collision/RR_shin_1.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
- link RR_thigh: mass 0.11726 -> 0.12481; geometry collision mesh filename=package://twist_2_0_description/meshes/collision/RR_thigh_0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; collision mesh filename=package://twist_2_0_description/meshes/collision/RR_thigh_1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
- link base_link: mass 0.39049 -> 0.40384; geometry collision mesh filename=package://twist_2_0_description/meshes/collision/base_link_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; collision mesh filename=package://twist_2_0_description/meshes/collision/base_link_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
Joints:
- joint FL_hip_pitch: limit lower=-2.6704 upper=1.0647 effort=1.91 velocity=4.71 -> lower=-2.1468 upper=1.0647 effort=1.91 velocity=4.71
- joint FL_hip_yaw: limit lower=-1.8675 upper=1.8675 effort=1.91 velocity=4.71 -> lower=-1.8675 upper=1.7977 effort=1.91 velocity=4.71; origin xyz=0.0810867 0.0810867 0 rpy=0 0 0 -> xyz=0.0809099 0.0809099 0 rpy=0 0 0
- joint FL_knee: limit lower=-0.8901 upper=3.1416 effort=1.91 velocity=4.71 -> lower=-0.8552 upper=3.1416 effort=1.91 velocity=4.71
- joint FR_hip_pitch: limit lower=-2.6704 upper=1.0647 effort=1.91 velocity=4.71 -> lower=-2.1468 upper=1.0647 effort=1.91 velocity=4.71
- joint FR_hip_yaw: limit lower=-1.8675 upper=1.8675 effort=1.91 velocity=4.71 -> lower=-1.8675 upper=1.7977 effort=1.91 velocity=4.71; origin xyz=0.0809099 -0.0809099 0 rpy=0 0 0 -> xyz=0.0810867 -0.0810867 0 rpy=0 0 0
- joint FR_knee: limit lower=-0.8901 upper=3.1416 effort=1.91 velocity=4.71 -> lower=-0.8552 upper=3.1416 effort=1.91 velocity=4.71
- joint RL_hip_pitch: limit lower=-2.6704 upper=1.0647 effort=1.91 velocity=4.71 -> lower=-2.1468 upper=1.0647 effort=1.91 velocity=4.71
- joint RL_hip_yaw: limit lower=-1.8675 upper=1.8675 effort=1.91 velocity=4.71 -> lower=-1.8675 upper=1.7977 effort=1.91 velocity=4.71
- joint RL_knee: limit lower=-0.8901 upper=3.1416 effort=1.91 velocity=4.71 -> lower=-0.8552 upper=3.1416 effort=1.91 velocity=4.71
- joint RR_hip_pitch: limit lower=-2.6704 upper=1.0647 effort=1.91 velocity=4.71 -> lower=-2.1468 upper=1.0647 effort=1.91 velocity=4.71
- joint RR_hip_yaw: limit lower=-1.8675 upper=1.8675 effort=1.91 velocity=4.71 -> lower=-1.8675 upper=1.7977 effort=1.91 velocity=4.71
- joint RR_knee: limit lower=-0.8901 upper=3.1416 effort=1.91 velocity=4.71 -> lower=-0.8552 upper=3.1416 effort=1.91 velocity=4.71
